Commit message: joystick working but rvizz is bugging

File: description/ros2_control.xacro (robot description, xacro)
@@ -4,61 +4,26 @@
         <ros2_control name="RealRobot" type="system">
             <hardware>
-                <!-- Plugin for controlling motors via Raspberry Pi GPIO for L298N -->
-                <plugin>rpi_gpio_control/L298NPlugin</plugin>
-                <param name="left_rear_wheel_name">left_rear_wheel_joint</param>
-                <param name="right_rear_wheel_name">right_rear_wheel_joint</param>
-                <param name="left_front_wheel_name">left_front_wheel_joint</param>
-                <param name="right_front_wheel_name">right_front_wheel_joint</param>
-                <!-- GPIO Pin Configuration for L298N Motor Driver -->
-                <!-- Left Rear Motor -->
-                <param name="left_rear_pwm_pin">18</param>   <!-- PWM pin for left rear wheel -->
-                <param name="left_rear_dir_pin">23</param>   <!-- Direction pin for left rear wheel -->
-                <!-- Right Rear Motor -->
-                <param name="right_rear_pwm_pin">19</param>   <!-- PWM pin for right rear wheel -->
-                <param name="right_rear_dir_pin">24</param>   <!-- Direction pin for right rear wheel -->
-                <!-- Left Front Motor -->
-                <param name="left_front_pwm_pin">12</param>  <!-- PWM pin for left front wheel -->
-                <param name="left_front_dir_pin">25</param>  <!-- Direction pin for left front wheel -->
-                <!-- Right Front Motor -->
-                <param name="right_front_pwm_pin">13</param>  <!-- PWM pin for right front wheel -->
-                <param name="right_front_dir_pin">26</param>  <!-- Direction pin for right front wheel -->
+                <plugin>diffdrive_arduino/DiffDriveArduinoHardware</plugin>
+                <param name="left_wheel_name">left_wheel_joint</param>
+                <param name="right_wheel_name">right_wheel_joint</param>
                 <param name="loop_rate">30</param>
-                <param name="timeout">1000</param>
+                <param name="device">/dev/serial/by-path/platform-fd500000.pcie-pci-0000:01:00.0-usb-0:1.3:1.0-port0</param>
+                <param name="baud_rate">57600</param>
+                <param name="timeout_ms">1000</param>
+                <param name="enc_counts_per_rev">3436</param>
+                <param name="pid_p">20</param>
+                <param name="pid_d">12</param>
+                <param name="pid_i">0</param>
+                <param name="pid_o">50</param>
             </hardware>
-            <!-- Rear Left Wheel -->
-            <joint name="left_rear_wheel_joint">
-                <command_interface name="velocity">
-                    <param name="min">-10</param>
-                    <param name="max">10</param>
-                </command_interface>
+            <joint name="${prefix}left_wheel_joint">
+                <command_interface name="velocity"/>
+                <state_interface name="position"/>
                 <state_interface name="velocity"/>
+            </joint>
+            <joint name="${prefix}right_wheel_joint">
+                <command_interface name="velocity"/>
                 <state_interface name="position"/>
-            </joint>
-            <!-- Rear Right Wheel -->
-            <joint name="right_rear_wheel_joint">
-                <command_interface name="velocity">
-                    <param name="min">-10</param>
-                    <param name="max">10</param>
-                </command_interface>
                 <state_interface name="velocity"/>
-                <state_interface name="position"/>
-            </joint>
-            <!-- Front Left Wheel -->
-            <joint name="left_front_wheel_joint">
-                <command_interface name="velocity">
-                    <param name="min">-10</param>
-                    <param name="max">10</param>
-                </command_interface>
-                <state_interface name="velocity"/>
-                <state_interface name="position"/>
-            </joint>
-            <!-- Front Right Wheel -->
-            <joint name="right_front_wheel_joint">
-                <command_interface name="velocity">
-                    <param name="min">-10</param>
-                    <param name="max">10</param>
-                </command_interface>
-                <state_interface name="velocity"/>
-                <state_interface name="position"/>
             </joint>
         </ros2_control>
